File: PCB/PCB.kicad_pcb (KiCad board)
At the start: 2 copper layers, 150 x 100 mm, 77 parts, among them J3 keys1_5, J4 keys6_12, J5 keys13_17, J6 keys18_24, J7 Conn_pen, J8 Conn_pen, SW1 PWR_SW, SW2 SW_Push, U1 74HC595D, U2 ATmega4809-A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

Commit message: Silkscreen
Parts:
- moved SW2 4.53 mm to (94.5, 34.5)
Routing:
- net Net-(BT1-Pad1): track 43.0 -> 0.00 mm
- net /SONG: track 48.3 -> 53.0 mm
- added copper zone on F.Cu, net Net-(BT1-Pad1)
Other:
- board text added: "1"
- board text added: "1. Last Christmas"
- board text added: "10"
- board text added: "10. Never Gonna Give You Up"
- board text added: "11. Super Mario"
- board text added: "12"
- board text added: "12. Imperial March"
- board text added: "2"
- board text added: "2. Jingle Bells"
- board text added: "3"
- board text added: "3. All I Want For Christmas Is You"
- board text added: "4"
- board text added: "4. Rockin Around The Christmas Tree"
- board text added: "5"
- board text added: "5. Feliz Navidad"
- board text added: "6"
- board text added: "6. We Wish You A Merry Christmas"
- board text added: "7"
- board text added: "7. Silent Night"
- board text added: "8"
- board text added: "8. Funky Town"
- board text added: "9"
- board text added: "9. Let's Groove"
- board text added: "Designed by: Daniel Quach Adam Anderson"
- board text added: "Hold button and touch pad with pen to select song"
- board text added: "Left side - Learn Right side - Auto"
- board text added: "Song select"
