File: PCB/PCB.kicad_pcb (KiCad board)
At the start: 2 copper layers, 150 x 100 mm, 77 parts, among them J3 keys1_5, J4 keys6_12, J5 keys13_17, J6 keys18_24, J7 Conn_pen, J8 Conn_pen, SW1 PWR_SW, SW2 SW_Push, U1 74HC595D, U2 ATmega4809-A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

Commit message: Finishing touches
Parts:
- added G***: LOGO, xmasLib:tree, B.Cu at (30.0, 50.0)
- added G***: LOGO, xmasLib:star, B.Cu at (53.5, 31.0)
- added G***: LOGO, xmasLib:star, B.Cu at (35.0, 44.0)
- added G***: LOGO, xmasLib:tree, B.Cu at (59.5, 44.0)
- added G***: LOGO, xmasLib:star, B.Cu at (70.0, 46.0)
- added G***: LOGO, xmasLib:tree, B.Cu at (44.0, 31.0)
- added G***: LOGO, xmasLib:star, B.Cu at (52.5, 43.0)
- added REF**: ToolingHole, xmasLib:ToolingHole, F.Cu at (102.5, 124.5)
- added REF**: ToolingHole, xmasLib:ToolingHole, F.Cu at (30.0, 29.5)
- added REF**: ToolingHole, xmasLib:ToolingHole, F.Cu at (170.0, 29.5)
- SW2: footprint Button_Switch_SMD:SW_Push_1P1T_NO_6x6mm_H9.5mm -> Button_Switch_SMD:SW_Push_1P1T_NO_CK_KSC6xxJ
Routing:
- net GND: track 212.2 -> 211.0 mm
Other:
- board text added: "JLCJLCJLCJLC"
