File: PCB/PCB.kicad_sch (KiCad schematic)
At the start: 6 parts

Commit message: schematic almost done
Parts:
- removed U? (x3): 74HC164, Package_SO:SOIC-14_3.9x8.7mm_P1.27mm, symbol 74xx:74HC164
- added C1, C3, C4, C5, C6: 100n, Capacitor_SMD:C_0603_1608Metric, symbol Device:C_Small
- added C2: 10u, Capacitor_SMD:C_0603_1608Metric, symbol Device:C_Small
- added D1, D10, D11, D12, D13, D14, D15, D16, D17, D18, D19, D2, D20, D21, D22, D23, D24, D3, D4, D5, D6, D7, D8, D9: LED, LED_SMD:LED_0603_1608Metric, symbol Device:LED_Small
- added J1: Conn_01x03, Connector_PinHeader_2.54mm:PinHeader_1x03_P2.54mm_Vertical, symbol Connector_Generic:Conn_01x03
- added JP1: RST_JP, Jumper:SolderJumper-2_P1.3mm_Open_RoundedPad1.0x1.5mm, symbol Jumper:SolderJumper_2_Open
- added R1, R10, R11, R12, R13, R14, R15, R16, R17, R18, R19, R2, R20, R21, R22, R23, R24, R3, R4, R5, R6, R7, R8, R9: 1k, Resistor_SMD:R_0603_1608Metric, symbol Device:R_Small
- added U1, U3, U4: 74HC595D, xmasLib:SOIC127P600X175-16N, symbol 74HC595D_118:74HC595D,118
- added U2: ATmega4809-A, Package_QFP:TQFP-48_7x7mm_P0.5mm, symbol MCU_Microchip_ATmega:ATmega4809-A
- gave numbers to parts that had none: 1
Connections:
- net +5V is gone; now on net +3V0: J2.3 (Pin_3)
- net +3V0: now also C1.2, C5.1, C6.2, U1.16 (VCC), U3.16 (VCC), U4.16 (VCC)
- net UPDI: now also U2.41 (UPDI)
- net PA2: now reaches BZ1.1 (-)
- net PA2: now also U2.46 (PA2)
- net GNDREF renamed GND
- net GND: now also C1.1, C2.2, C3.2, C4.2, C5.2, C6.1, D1.1 (K), D10.1 (K), D11.1 (K), D12.1 (K), D13.1 (K), D14.1 (K), D15.1 (K), D16.1 (K), D17.1 (K), D18.1 (K), D19.1 (K), D2.1 (K), D20.1 (K), D21.1 (K), D22.1 (K), D23.1 (K), D24.1 (K), D3.1 (K), D4.1 (K), D5.1 (K), D6.1 (K), D7.1 (K), D8.1 (K), D9.1 (K), J1.3 (Pin_3), JP1.1 (A), U1.8 (GND), U2.15 (GND), U2.29 (GND), U2.43 (GND), U3.8 (GND), U4.8 (GND)
- new net: R6.1, U1.5 (Q5)
- new net: D6.2 (A), R6.2
- new net: R13.1, U3.4 (Q4)
- new net: D13.2 (A), R13.2
- new net: D9.2 (A), R9.2
- new net: R2.1, U1.1 (Q1)
- new net: R1.1, U1.15 (Q0)
- new net: R3.1, U1.2 (Q2)
- new net: R4.1, U1.3 (Q3)
- new net: R5.1, U1.4 (Q4)
- new net: R7.1, U1.6 (Q6)
- new net: R8.1, U1.7 (Q7)
- new net: U1.9 (Q7_2), U3.14 (DS)
- new net: R21.1, U4.4 (Q4)
- new net: D21.2 (A), R21.2
- new net: D2.2 (A), R2.2
- new net: D12.2 (A), R12.2
- new net: D5.2 (A), R5.2
- new net: D16.2 (A), R16.2
- new net: D8.2 (A), R8.2
- new net: C2.1, C3.1, C4.1, U2.14 (VCC), U2.28 (AVCC), U2.42 (VCC)
- new net: D3.2 (A), R3.2
- new net: R15.1, U3.6 (Q6)
- new net: D15.2 (A), R15.2
- new net: R10.1, U3.1 (Q1)
- new net: D10.2 (A), R10.2
- new net: D17.2 (A), R17.2
- new net: D4.2 (A), R4.2
- new net: R20.1, U4.3 (Q3)
- new net: D20.2 (A), R20.2
- new net: R9.1, U3.15 (Q0)
- new net: D19.2 (A), R19.2
- new net: D7.2 (A), R7.2
- new net: D18.2 (A), R18.2
- new net: R16.1, U3.7 (Q7)
- new net: R17.1, U4.15 (Q0)
- new net: R11.1, U3.2 (Q2)
- new net: R12.1, U3.3 (Q3)
- new net: R14.1, U3.5 (Q5)
- new net: U3.9 (Q7_2), U4.14 (DS)
- new net: R22.1, U4.5 (Q5)
- new net: D22.2 (A), R22.2
- new net: D11.2 (A), R11.2
- new net: R24.1, U4.7 (Q7)
- new net: D24.2 (A), R24.2
- new net: D1.2 (A), R1.2
- new net: D14.2 (A), R14.2
- new net: R23.1, U4.6 (Q6)
- new net: D23.2 (A), R23.2
- new net: R18.1, U4.1 (Q1)
- new net: R19.1, U4.2 (Q2)
- new net PA0/TX: J1.1 (Pin_1), U2.44 (PA0)
- new net PA1/RX: J1.2 (Pin_2), U2.45 (PA1)
- new net PF6/~{RST}: JP1.2 (B), U2.40 (PF6/~{RESET})
- new net SER: U1.14 (DS)
- new net SH_C: U1.11 (SH_CP), U3.11 (SH_CP), U4.11 (SH_CP)
- new net ST_C: U1.12 (ST_CP), U3.12 (ST_CP), U4.12 (ST_CP)
- new net ~{OE}: U1.13 (~OE), U3.13 (~OE), U4.13 (~OE)
- new net ~{RST}: U1.10 (~MR), U3.10 (~MR), U4.10 (~MR)
- no-connect marks 0 -> 1
Other:
- note added: "Need to be assigned"
- moved on the sheet: BT1, BZ1, J2

Commit message: Update PCB.kicad_sch
Parts:
- added SW?: SW_SPDT, symbol Switch:SW_SPDT
Connections:
- net +3V0: now also SW?.2 (B); no longer BT1.1 (+)
- new net: BT1.1 (+), SW?.1 (A)
Other:
- moved on the sheet: BT1, J1, J2, JP1

Commit message: Rough placement of components done
Parts:
- added J3: keys1_5, xmasLib:3w2b, symbol Connector_Generic:Conn_01x05
- added J4: keys6_12, xmasLib:4w3b, symbol Connector_Generic:Conn_01x07
- added J5: keys13_17, xmasLib:3w2b, symbol Connector_Generic:Conn_01x05
- added J6: keys18_24, xmasLib:4w3b, symbol Connector_Generic:Conn_01x07
- J1: value Conn_01x03 -> Serial_3P
- J2: value Conn_01x03_Male -> UPDI_3P
- SW1: renamed from SW?; value SW_SPDT -> PWR_SW; footprint (none) -> Button_Switch_SMD:SW_SPDT_CK-JS102011SAQN
Connections:
- net +3V0: now also C2.1, C3.1, C4.1, U2.14 (VCC), U2.28 (AVCC), U2.42 (VCC)
- no-connect marks 1 -> 2
Other:
- note added: "Add stylophone pen connector"
Changed lines of the file:
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@@
   )
   (no_connect (at 209.55 247.65))
+  (no_connect (at 214.63 60.96))
   (wire (pts (xy 76.2 242.57) (xy 82.55 242.57))
     (stroke (width 0) (type default) (color 0 0 0 0))
@@
     (stroke (width 0) (type default) (color 0 0 0 0))
   )
+  (wire (pts (xy 77.47 24.13) (xy 77.47 27.94))
+    (stroke (width 0) (type default) (color 0 0 0 0))
+  )
   (wire (pts (xy 87.63 227.33) (xy 87.63 229.87))
     (stroke (width 0) (type default) (color 0 0 0 0))
@@
   )
   (text "Need to be assigned\n" (at 21.59 208.28 0)
+    (effects (font (size 1.27 1.27)) (justify left bottom))
+  )
+  (text "Add stylophone pen connector" (at 237.49 106.68 0)
     (effects (font (size 1.27 1.27)) (justify left bottom))
   )
@@
     )
     (property "Datasheet" "" (id 3) (at 158.75 245.11 0)
+      (effects (font (size 1.27 1.27)) hide)
+    )
+    (pin "1")
+  )
+  (symbol (lib_id "power:+3V0") (at 77.47 24.13 0) (unit 1)
+    (in_bom yes) (on_board yes) (fields_autoplaced)
+    (property "Reference" "#PWR018" (id 0) (at 77.47 27.94 0)
+      (effects (font (size 1.27 1.27)) hide)
+    )
+    (property "Value" "+3V0" (id 1) (at 77.47 20.5255 0))
+    (property "Footprint" "" (id 2) (at 77.47 24.13 0)
+      (effects (font (size 1.27 1.27)) hide)
+    )
+    (property "Datasheet" "" (id 3) (at 77.47 24.13 0)
       (effects (font (size 1.27 1.27)) hide)
     )
@@
     (pin "1")
   )
+  (symbol (lib_id "Connector_Generic:Conn_01x07") (at 184.15 154.94 90) (mirror x) (unit 1)
+    (in_bom yes) (on_board yes)
+    (property "Reference" "J6" (id 0) (at 185.42 157.48 90)
+      (effects (font (size 1.27 1.27)) (justify left))
+    )
+    (property "Value" "keys18_24" (id 1) (at 189.23 160.02 90)
+      (effects (font (size 1.27 1.27)) (justify left))
+    )
+    (property "Footprint" "xmasLib:4w3b" (id 2) (at 184.15 154.94 0)
+      (effects (font (size 1.27 1.27)) hide)
+    )
+    (property "Datasheet" "~" (id 3) (at 184.15 154.94 0)
+      (effects (font (size 1.27 1.27)) hide)
+    )
+    (pin "1")
+    (pin "2")
+    (pin "3")
+    (pin "4")
+    (pin "5")
+    (pin "6")
+    (pin "7")
+  )
   (symbol (lib_id "Device:LED_Small") (at 85.09 245.11 180) (unit 1)
     (in_bom yes) (on_board yes)
@@
   (symbol (lib_id "Switch:SW_SPDT") (at 217.17 55.88 270) (unit 1)
     (in_bom yes) (on_board yes) (fields_autoplaced)
-    (property "Reference" "SW?" (id 0) (at 220.98 54.6099 90)
-      (effects (font (size 1.27 1.27)) (justify left))
-    )
-    (property "Value" "SW_SPDT" (id 1) (at 220.98 57.1499 90)
-      (effects (font (size 1.27 1.27)) (justify left))
-    )
-    (property "Footprint" "" (id 2) (at 217.17 55.88 0)
+    (property "Reference" "SW1" (id 0) (at 220.98 54.6099 90)
+      (effects (font (size 1.27 1.27)) (justify left))
+    )
+    (property "Value" "PWR_SW" (id 1) (at 220.98 57.1499 90)
+      (effects (font (size 1.27 1.27)) (justify left))
+    )
+    (property "Footprint" "Button_Switch_SMD:SW_SPDT_CK-JS102011SAQN" (id 2) (at 217.17 55.88 0)
       (effects (font (size 1.27 1.27)) hide)
     )
@@
     (pin "2")
   )
+  (symbol (lib_id "Connector_Generic:Conn_01x07") (at 148.59 154.94 90) (mirror x) (unit 1)
+    (in_bom yes) (on_board yes)
+    (property "Reference" "J4" (id 0) (at 149.86 157.48 90)
+      (effects (font (size 1.27 1.27)) (justify left))
+    )
+    (property "Value" "keys6_12" (id 1) (at 152.4 160.02 90)
+      (effects (font (size 1.27 1.27)) (justify left))
+    )
+    (property "Footprint" "xmasLib:4w3b" (id 2) (at 148.59 154.94 0)
+      (effects (font (size 1.27 1.27)) hide)
+    )
+    (property "Datasheet" "~" (id 3) (at 148.59 154.94 0)
+      (effects (font (size 1.27 1.27)) hide)
+    )
+    (pin "1")
+    (pin "2")
+    (pin "3")
+    (pin "4")
+    (pin "5")
+    (pin "6")
+    (pin "7")
+  )
   (symbol (lib_id "Device:R_Small") (at 215.9 242.57 90) (unit 1)
     (in_bom yes) (on_board yes)
@@
       (effects (font (size 1.27 1.27)) (justify left))
     )
-    (property "Value" "Conn_01x03" (id 1) (at 269.24 88.8999 0)
+    (property "Value" "Serial_3P" (id 1) (at 269.24 88.8999 0)
       (effects (font (size 1.27 1.27)) (justify left))
     )
@@
   (symbol (lib_id "Device:C_Small") (at 170.18 219.71 180) (unit 1)
     (in_bom yes) (on_board yes)
-    (property "Reference" "C6" (id 0) (at 166.37 218.44 0)
+    (property "Reference" "C6" (id 0) (at 165.1 218.44 0)
       (effects (font (size 1.27 1.27)) (justify right))
     )
@@
     (pin "2")
   )
+  (symbol (lib_id "Connector_Generic:Conn_01x05") (at 130.81 154.94 90) (mirror x) (unit 1)
+    (in_bom yes) (on_board yes)
+    (property "Reference" "J3" (id 0) (at 132.08 157.48 90)
+      (effects (font (size 1.27 1.27)) (justify left))
+    )
+    (property "Value" "keys1_5" (id 1) (at 134.62 160.02 90)
+      (effects (font (size 1.27 1.27)) (justify left))
+    )
+    (property "Footprint" "xmasLib:3w2b" (id 2) (at 130.81 154.94 0)
+      (effects (font (size 1.27 1.27)) hide)
+    )
+    (property "Datasheet" "~" (id 3) (at 130.81 154.94 0)
+      (effects (font (size 1.27 1.27)) hide)
+    )
+    (pin "1")
+    (pin "2")
+    (pin "3")
+    (pin "4")
+    (pin "5")
+  )
   (symbol (lib_id "Device:C_Small") (at 68.58 30.48 0) (unit 1)
     (in_bom yes) (on_board yes) (fields_autoplaced)
@@
   (symbol (lib_id "Connector:Conn_01x03_Male") (at 266.7 41.91 180) (unit 1)
     (in_bom yes) (on_board yes) (fields_autoplaced)
-    (property "Reference" "J2" (id 0) (at 267.4112 41.0015 0)
+    (property "Reference" "J2" (id 0) (at 267.97 40.6399 0)
       (effects (font (size 1.27 1.27)) (justify right))
     )
-    (property "Value" "Conn_01x03_Male" (id 1) (at 267.4112 43.7766 0)
+    (property "Value" "UPDI_3P" (id 1) (at 267.97 43.1799 0)
       (effects (font (size 1.27 1.27)) (justify right))
     )
@@
     (pin "2")
     (pin "3")
+  )
+  (symbol (lib_id "Connector_Generic:Conn_01x05") (at 166.37 154.94 90) (mirror x) (unit 1)
+    (in_bom yes) (on_board yes)
+    (property "Reference" "J5" (id 0) (at 166.37 157.48 90))
+    (property "Value" "keys13_17" (id 1) (at 166.37 160.02 90))
+    (property "Footprint" "xmasLib:3w2b" (id 2) (at 166.37 154.94 0)
+      (effects (font (size 1.27 1.27)) hide)
+    )
+    (property "Datasheet" "~" (id 3) (at 166.37 154.94 0)
+      (effects (font (size 1.27 1.27)) hide)
+    )
+    (pin "1")
+    (pin "2")
+    (pin "3")
+    (pin "4")
+    (pin "5")
   )
   (symbol (lib_id "Device:LED_Small") (at 227.33 242.57 180) (unit 1)
@@
       (reference "#PWR017") (unit 1) (value "GND") (footprint "")
     )
+    (path "/1d618fb2-efc3-4996-ab77-9be4a3955fa9"
+      (reference "#PWR018") (unit 1) (value "+3V0") (footprint "")
+    )
     (path "/d7c96d03-c33d-42a4-b9f5-33ebc94d6064"
       (reference "BT1") (unit 1) (value "Battery_Cell") (footprint "xmasLib:BAT-HLD-001")
@@
     )
     (path "/bf012aef-fa62-4572-adfe-b9060c5749c6"
-      (reference "J1") (unit 1) (value "Conn_01x03") (footprint "Connector_PinHeader_2.54mm:PinHeader_1x03_P2.54mm_Vertical")
+      (reference "J1") (unit 1) (value "Serial_3P") (footprint "Connector_PinHeader_2.54mm:PinHeader_1x03_P2.54mm_Vertical")
     )
     (path "/f815fa82-71e8-446f-ac86-3883d2afcdf7"
-      (reference "J2") (unit 1) (value "Conn_01x03_Male") (footprint "Connector_PinHeader_2.54mm:PinHeader_1x03_P2.54mm_Vertical")
+      (reference "J2") (unit 1) (value "UPDI_3P") (footprint "Connector_PinHeader_2.54mm:PinHeader_1x03_P2.54mm_Vertical")
+    )
+    (path "/eb7a84b1-b974-4746-b629-74149a9b76bb"
+      (reference "J3") (unit 1) (value "keys1_5") (footprint "xmasLib:3w2b")
+    )
+    (path "/bde222bb-f90c-4b1d-8a7e-0adead7cda65"
+      (reference "J4") (unit 1) (value "keys6_12") (footprint "xmasLib:4w3b")
+    )
+    (path "/f8586a7a-9397-4f17-aed5-6ffc3b97403e"
+      (reference "J5") (unit 1) (value "keys13_17") (footprint "xmasLib:3w2b")
+    )
+    (path "/33194efc-ceab-4864-9cfd-99d9d0f5506b"
+      (reference "J6") (unit 1) (value "keys18_24") (footprint "xmasLib:4w3b")
     )
     (path "/87f71c26-7128-47dd-8641-9283fea19148"
@@
     )
     (path "/83084c48-2506-4438-9f06-1cc23b3d4759"
-      (reference "SW?") (unit 1) (value "SW_SPDT") (footprint "")
+      (reference "SW1") (unit 1) (value "PWR_SW") (footprint "Button_Switch_SMD:SW_SPDT_CK-JS102011SAQN")
     )
     (path "/18b77920-d592-4833-aaae-7c8641a646e3"

Commit message: Start routing
Parts:
- added J7: Conn_pen, Connector_PinHeader_2.54mm:PinHeader_1x01_P2.54mm_Vertical, symbol Connector_Generic:Conn_01x01
- added R25: ?, Resistor_SMD:R_0603_1608Metric, symbol Device:R_Small
- added SW2: SW_Push, Button_Switch_SMD:SW_Push_1P1T_NO_6x6mm_H9.5mm, symbol Switch:SW_Push
- J3, J5: footprint xmasLib:3w2b -> xmasLib:3w2bv2
- J4, J6: footprint xmasLib:4w3b -> xmasLib:4w3bv2
Connections:
- net GND: now also R25.1, SW2.2
- net PC0: now reaches U2.10 (PC0)
- net PC0: now also J4.1 (Pin_1)
- net PC1: now reaches U2.11 (PC1)
- net PC1: now also J3.5 (Pin_5)
- net PC2: now reaches U2.12 (PC2)
- net PC2: now also J3.4 (Pin_4)
- net PC3: now reaches U2.13 (PC3)
- net PC3: now also J3.3 (Pin_3)
- net PC4: now reaches U2.16 (PC4)
- net PC4: now also J3.2 (Pin_2)
- net PC5: now reaches U2.17 (PC5)
- net PC5: now also J3.1 (Pin_1)
- net PC6: now reaches U2.18 (PC6)
- net PC7: now reaches U2.19 (PC7)
- net PD0: now reaches U2.20 (PD0)
- net PD1: now reaches U2.21 (PD1)
- net PD2: now reaches U2.22 (PD2)
- net PD3: now reaches U2.23 (PD3)
- net PD3: now also J6.7 (Pin_7)
- net PD4: now reaches U2.24 (PD4)
- net PD4: now also J6.6 (Pin_6)
- net PD5: now reaches U2.25 (PD5)
- net PD5: now also J6.5 (Pin_5)
- net PD6: now reaches U2.26 (PD6)
- net PD6: now also J6.4 (Pin_4)
- net PD7: now reaches U2.27 (PD7)
- net PD7: now also J6.3 (Pin_3)
- net PE0: now reaches U2.30 (PE0)
- net PE0: now also J6.2 (Pin_2)
- net PE1: now reaches U2.31 (PE1)
- net PE1: now also J6.1 (Pin_1)
- net PE2: now reaches U2.32 (PE2)
- net PE2: now also J5.5 (Pin_5)
- net PE3: now reaches U2.33 (PE3)
- net PE3: now also J5.4 (Pin_4)
- net PF0: now reaches U2.34 (PF0)
- net PF0: now also J5.3 (Pin_3)
- net PF1: now reaches U2.35 (PF1)
- net PF1: now also J5.2 (Pin_2)
- net PF2: now reaches U2.36 (PF2)
- net PF2: now also J5.1 (Pin_1)
- net PB0: now reaches U2.4 (PB0)
- net PB0: now also J4.7 (Pin_7)
- net PB1: now reaches U2.5 (PB1)
- net PB1: now also J4.6 (Pin_6)
- net PB2: now reaches U2.6 (PB2)
- net PB2: now also J4.5 (Pin_5)
- net PB3: now reaches U2.7 (PB3)
- net PB3: now also J4.4 (Pin_4)
- net PB4: now reaches U2.8 (PB4)
- net PB4: now also J4.3 (Pin_3)
- net PB5: now reaches U2.9 (PB5)
- net PB5: now also J4.2 (Pin_2)
- new net: J7.1 (Pin_1), R25.2
Other:
- note added: "Song selection"

Commit message: Routing, pin assignments
Parts:
- removed JP1: RST_JP, Jumper:SolderJumper-2_P1.3mm_Open_RoundedPad1.0x1.5mm, symbol Jumper:SolderJumper_2_Open
- added TP1: Reset, TestPoint:TestPoint_Pad_D2.0mm, symbol Connector:TestPoint
- R25: value ? -> 1K
Connections:
- net SER is gone; now on net PC6: U1.14 (DS)
- net SH_C is gone; now on net PD1: U1.11 (SH_CP), U3.11 (SH_CP), U4.11 (SH_CP)
- net ST_C is gone; now on net PD0: U1.12 (ST_CP), U3.12 (ST_CP), U4.12 (ST_CP)
- net ~{OE} is gone; now on net PC7: U1.13 (~OE), U3.13 (~OE), U4.13 (~OE)
- net ~{RST} is gone; now on net PD2: U1.10 (~MR), U3.10 (~MR), U4.10 (~MR)
- net PB0: now also J4.4 (Pin_4); no longer J4.7 (Pin_7)
- net PB1: now also J4.3 (Pin_3); no longer J4.6 (Pin_6)
- net PB2: now also J4.2 (Pin_2); no longer J4.5 (Pin_5)
- net PB3: now also J4.1 (Pin_1); no longer J4.4 (Pin_4)
- net PB4: now also J3.5 (Pin_5); no longer J4.3 (Pin_3)
- net PB5: now also J3.4 (Pin_4); no longer J4.2 (Pin_2)
- net PC0: now also J3.3 (Pin_3); no longer J4.1 (Pin_1)
- net PC1: now also J3.2 (Pin_2); no longer J3.5 (Pin_5)
- net PC2: now also J3.1 (Pin_1); no longer J3.4 (Pin_4)
- net PF6/~{RST}: now also TP1.1
- net PA5: now reaches U2.1 (PA5)
- net PA5: now also J4.7 (Pin_7)
- net PA6: now reaches U2.2 (PA6)
- net PA6: now also J4.6 (Pin_6)
- net PA7: now reaches U2.3 (PA7)
- net PA7: now also J4.5 (Pin_5)
- net SONG: now reaches U2.37 (PF3)
- net SONG: now also SW2.1
- net PC3: no longer names the net of U2.13 (PC3)
- net PC3: no longer J3.3 (Pin_3)
- net PC4: no longer names the net of U2.16 (PC4)
- net PC4: no longer J3.2 (Pin_2)
- net PC5: no longer names the net of U2.17 (PC5)
- net PC5: no longer J3.1 (Pin_1)

Commit message: Final routing
Parts:
- removed J1: Serial_3P, Connector_PinHeader_2.54mm:PinHeader_1x03_P2.54mm_Vertical, symbol Connector_Generic:Conn_01x03
- removed J2: UPDI_3P, Connector_PinHeader_2.54mm:PinHeader_1x03_P2.54mm_Vertical, symbol Connector:Conn_01x03_Male
- added J8: Conn_pen, MountingHole:MountingHole_2.2mm_M2_Pad_Via, symbol Connector_Generic:Conn_01x01
- added TP2, TP3, TP4, TP5, TP6, TP7: TestPoint_Small, TestPoint:TestPoint_Pad_D1.5mm, symbol Connector:TestPoint_Small
- J7: footprint Connector_PinHeader_2.54mm:PinHeader_1x01_P2.54mm_Vertical -> MountingHole:MountingHole_2.2mm_M2_Pad_Via
Connections:
- net +3V0: now also TP2.1
- net GND: now also TP4.1, TP7.1
- net PA0/TX: now also TP5.1
- net PA1/RX: now also TP6.1
- net UPDI: now also TP3.1
- net at J7.1 (Pin_1), R25.2: now also J8.1 (Pin_1)

Commit message: Finishing touches
Parts:
- SW2: footprint Button_Switch_SMD:SW_Push_1P1T_NO_6x6mm_H9.5mm -> Button_Switch_SMD:SW_Push_1P1T_NO_CK_KSC6xxJ
Changed lines of the file:
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@@
     (property "Reference" "SW2" (id 0) (at 185.42 28.6725 0))
     (property "Value" "SW_Push" (id 1) (at 185.42 31.4476 0))
-    (property "Footprint" "Button_Switch_SMD:SW_Push_1P1T_NO_6x6mm_H9.5mm" (id 2) (at 185.42 30.48 0)
+    (property "Footprint" "Button_Switch_SMD:SW_Push_1P1T_NO_CK_KSC6xxJ" (id 2) (at 185.42 30.48 0)
       (effects (font (size 1.27 1.27)) hide)
     )
@@
     )
     (path "/e8263da8-e2fb-43a9-a299-174a84b3346a"
-      (reference "SW2") (unit 1) (value "SW_Push") (footprint "Button_Switch_SMD:SW_Push_1P1T_NO_6x6mm_H9.5mm")
+      (reference "SW2") (unit 1) (value "SW_Push") (footprint "Button_Switch_SMD:SW_Push_1P1T_NO_CK_KSC6xxJ")
     )
     (path "/fdb8ea48-5fca-4d7c-94ba-c5c2ee68cff2"
